Commit message: hardware

File: src/ned-ros2-driver/niryo_ned_moveit_configs/niryo_ned2_dual_gripper_moveit_config/config/niryo_ned2_dual_arm.ros2_control.xacro (robot description, xacro)
@@ -92,16 +92,4 @@
                 </state_interface>
             </joint>
-            <joint name="arm_2_joint_base_to_mors_1">
-                <command_interface name="position"/>
-                <state_interface name="position">
-                  <param name="initial_value">${initial_positions['arm_2_joint_base_to_mors_1']}</param>
-                </state_interface>
-            </joint>
-            <joint name="arm_2_joint_base_to_mors_2">
-                <command_interface name="position"/>
-                <state_interface name="position">
-                  <param name="initial_value">${initial_positions['arm_2_joint_base_to_mors_2']}</param>
-                </state_interface>
-            </joint>
         </ros2_control>
     </xacro:macro>
